File: Hornbill_PCB/Hornbill.sch (KiCad schematic (older format))
At the start: 69 parts, among them P1 CONN_01X19, P10 CONN_01X03, P11 CONN_01X03, P12 CONN_01X19, P13 CONN_01X03, P14 CONN_01X09, P15 CONN_01X09, P16 CONN_01X09, P17 CONN_01X09, P18 CONN_01X09, P19 CONN_01X09, P2 CONN_01X19, P20 CONN_01X09, P21 CONN_01X09, P22 CONN_01X09, P23 CONN_01X09, P24 CONN_01X09, P25 CONN_01X13, P26 CONN_01X13, P27 CONN_01X13, P28 CONN_01X13, P29 CONN_01X09, P3 CONN_01X19, P30 CONN_01X09, P4 CONN_01X19, P5 CONN_01X19, P6 CONN_01X19, P7 CONN_01X03, P8 CONN_01X19, P9 CONN_01X03, Q1 Q_NPN_BCE, U1 SHT31_DIS, U2 SD_Crard, U3 RGB_4pin, U4 ESP32_Breakout1, U5 MountingHole, U6 MountingHole, U7 MountingHole, U8 MountingHole

Commit message: PCB layout routing completed
Parts:
- removed U1: SHT31_DIS, ee:SHT31_DIS, symbol SHT31_DIS
- added R22: 0r, Resistors_SMD:R_0603_HandSoldering, symbol R-RESCUE-Hornbill
- added RH1: SHT31-DIS, nosuz lib:DFN-8_SHT-3x-DIS, symbol SHT31-DIS
- C1: value 100nF -> 10uF
Connections:
- net +5V: now also R22.2
- net 3.3V: now also RH1.5 (VDD)
- net GND: now also RH1.7 (R), RH1.8 (VSS), RH1.9 (pad)
- net SCL: now also RH1.4 (SCL)
- net SDA: now also RH1.1 (SDA)
- net at R2.1: now also RH1.2 (ADDR)
- net at R1.1: now also RH1.6 (nRESET)
- net at P7.3 (P3), R21.2: now also R22.1
Other:
- note added: "Hornbill ESP32"
- note removed: "Hornbill Base Board"
- moved on the sheet: P7, R10, R11, R12, R13, R14, R2, R21, R9, U3, U5, U6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

Commit message: Chnges done as per issues
Parts:
- removed D3, D4: LED, LEDs:LED-3MM, symbol LED-RESCUE-Hornbill
- removed Q1: Q_NPN_BCE, ee:SOT_23, symbol Q_NPN_BCE
- removed R15: 10k, Resistors_SMD:R_0603_HandSoldering, symbol R-RESCUE-Hornbill
- removed R16: 10K, Resistors_SMD:R_0603_HandSoldering, symbol R-RESCUE-Hornbill
- removed R17: 1K, Resistors_SMD:R_0603_HandSoldering, symbol R-RESCUE-Hornbill
- removed R18, R19: 33K, Resistors_SMD:R_0603_HandSoldering, symbol R-RESCUE-Hornbill
- added P31, P32, P33, P34: CONN_01X03, Pin_Headers:Pin_Header_Straight_1x03_Pitch2.54mm, symbol CONN_01X03
- added Q1: Q_NPN_BEC, EE:SOT_23, symbol Q_NPN_BEC
Connections:
- net B: now also P4.9 (P9), U4.30 (27); no longer P3.9 (P9), U4.9 (17)
- net G: now also P4.10 (P10), U4.29 (26); no longer P3.7 (P7), U4.7 (4)
- net GND: now also U2.3 (CMD), Q1.2 (E)
- net R: now also P4.11 (P11), U4.28 (25); no longer P3.6 (P6), U4.6 (0)
- net at D1.1 (K): now also D5.2 (A)
- net at D2.1 (K): now also D6.2 (A)
- net at R3.1: now also Q1.1 (B)
- net at R7.2: now also Q1.3 (C)
- net IO5: now reaches U2.1 (DATA2)
- net IO5: now also P3.10 (P10), U4.10 (5)
- net CLK renamed IO18
- net MISO renamed IO19
- net MOSI renamed IO23
- net IO23: now also U2.2 (CD/DATA3); no longer U2.3 (CMD)
- net SD_DTCT: no longer names the net of P3.3 (P3), U4.3 (SD1)
- net SD_DTCT: no longer U2.9 (CD)
- net SSEL: no longer names the net of P3.5 (P5), U4.5 (2)
- net SSEL: no longer U2.2 (CD/DATA3)
- new net: P3.6 (P6), U4.6 (0)
- new net: P3.7 (P7), U4.7 (4)
- new net: P3.9 (P9), U4.9 (17)
- no-connect marks 296 -> 311
Changed lines of the file:
@@
 LIBS:contrib
 LIBS:valves
-LIBS:nosuz
+LIBS:MCU_BaseBoard-cache
+LIBS:ExploreM3-cache
 LIBS:Hornbill-cache
 EELAYER 25 0
@@
 $EndComp
 $Comp
-L LED-RESCUE-Hornbill D3
-U 1 1 58627710
-P 9300 1250
-F 0 "D3" H 9300 1350 50  0000 C CNN
-F 1 "LED" H 9300 1150 50  0000 C CNN
-F 2 "LEDs:LED-3MM" H 9300 1250 50  0001 C CNN
-F 3 "" H 9300 1250 50  0000 C CNN
-	1    9300 1250
-	-1   0    0    1
-$EndComp
-$Comp
 L LED-RESCUE-Hornbill D5
 U 1 1 58627769
@@
 $EndComp
 $Comp
-L LED-RESCUE-Hornbill D4
-U 1 1 58627824
-P 9300 1700
-F 0 "D4" H 9300 1800 50  0000 C CNN
-F 1 "LED" H 9300 1600 50  0000 C CNN
-F 2 "LEDs:LED-3MM" H 9300 1700 50  0001 C CNN
-F 3 "" H 9300 1700 50  0000 C CNN
-	1    9300 1700
-	-1   0    0    1
-$EndComp
-$Comp
 L LED-RESCUE-Hornbill D6
 U 1 1 58627882
@@
 $EndComp
 $Comp
-L Q_NPN_BCE Q1
-U 1 1 58627FE4
-P 10550 2600
-F 0 "Q1" H 10850 2650 50  0000 R CNN
-F 1 "Q_NPN_BCE" H 11150 2550 50  0000 R CNN
-F 2 "ee:SOT_23" H 10750 2700 50  0001 C CNN
-F 3 "" H 10550 2600 50  0000 C CNN
-	1    10550 2600
-	1    0    0    -1
-$EndComp
-$Comp
 L R-RESCUE-Hornbill R7
 U 1 1 58628161
@@
 $EndComp
 $Comp
-L R-RESCUE-Hornbill R18
-U 1 1 5864B0DF
-P 3900 5750
-F 0 "R18" V 3980 5750 50  0000 C CNN
-F 1 "33K" V 3900 5750 50  0000 C CNN
-F 2 "Resistors_SMD:R_0603_HandSoldering" V 3830 5750 50  0001 C CNN
-F 3 "" H 3900 5750 50  0000 C CNN
-	1    3900 5750
-	0    1    1    0
-$EndComp
-$Comp
-L R-RESCUE-Hornbill R19
-U 1 1 5864B358
-P 3900 6000
-F 0 "R19" V 3980 6000 50  0000 C CNN
-F 1 "33K" V 3900 6000 50  0000 C CNN
-F 2 "Resistors_SMD:R_0603_HandSoldering" V 3830 6000 50  0001 C CNN
-F 3 "" H 3900 6000 50  0000 C CNN
-	1    3900 6000
-	0    1    1    0
-$EndComp
-$Comp
 L GND #PWR06
 U 1 1 5864BCDA
@@
 	1    0    0    -1
 $EndComp
-$Comp
-L R-RESCUE-Hornbill R17
-U 1 1 5864C015
-P 2050 6200
-F 0 "R17" V 2130 6200 50  0000 C CNN
-F 1 "1K" V 2050 6200 50  0000 C CNN
-F 2 "Resistors_SMD:R_0603_HandSoldering" V 1980 6200 50  0001 C CNN
-F 3 "" H 2050 6200 50  0000 C CNN
-	1    2050 6200
-	0    1    1    0
-$EndComp
-$Comp
-L R-RESCUE-Hornbill R16
-U 1 1 5864D0FB
-P 1300 5450
-F 0 "R16" V 1380 5450 50  0000 C CNN
-F 1 "10K" V 1300 5450 50  0000 C CNN
-F 2 "Resistors_SMD:R_0603_HandSoldering" V 1230 5450 50  0001 C CNN
-F 3 "" H 1300 5450 50  0000 C CNN
-	1    1300 5450
-	1    0    0    -1
-$EndComp
-$Comp
-L R-RESCUE-Hornbill R15
-U 1 1 5864D1A9
-P 1050 5450
-F 0 "R15" V 1130 5450 50  0000 C CNN
-F 1 "10k" V 1050 5450 50  0000 C CNN
-F 2 "Resistors_SMD:R_0603_HandSoldering" V 980 5450 50  0001 C CNN
-F 3 "" H 1050 5450 50  0000 C CNN
-	1    1050 5450
-	1    0    0    -1
-$EndComp
 Text GLabel 8250 1400 1    47   Input ~ 0
 +5V
-Text GLabel 1050 5200 1    40   Input ~ 0
-3.3V
 $Comp
 L C-RESCUE-Hornbill C2
@@
 Text Label 2490 1850 0    40   ~ 0
 SDA
-Text Label 2450 5700 2    40   ~ 0
-SSEL
-Text Label 2450 5800 2    40   ~ 0
-MOSI
-Text Label 2450 5900 2    40   ~ 0
-CLK
-Text Label 2450 6000 2    40   ~ 0
-MISO
 Text GLabel 2100 4850 1    40   Input ~ 0
-3.3V
-Text GLabel 4200 5400 1    40   Input ~ 0
-3.3V
-Text GLabel 1650 6200 0    40   Input ~ 0
 3.3V
 Text Label 770  4070 2    40   ~ 0
@@
 Text Label 5400 2500 2    40   ~ 0
 SDA
-Text Label 5400 1600 2    40   ~ 0
-SSEL
-Text Label 5400 2900 2    40   ~ 0
-MOSI
-Text Label 5400 2200 2    40   ~ 0
-CLK
-Text Label 5400 2300 2    40   ~ 0
-MISO
-Text Label 5400 1400 2    40   ~ 0
-SD_DTCT
-Text Label 2450 6100 2    40   ~ 0
-SD_DTCT
 Text GLabel 850  1100 1    40   Input ~ 0
 3.3V
@@
 Text Label 8900 2600 2    40   ~ 0
 IR_Tx
-Text Label 5400 1700 2    40   ~ 0
+Text Label 6600 2200 0    40   ~ 0
 R
-Text Label 5400 1800 2    40   ~ 0
+Text Label 6600 2100 0    40   ~ 0
 G
-Text Label 5400 2000 2    40   ~ 0
+Text Label 6600 2000 0    40   ~ 0
 B
 Text Label 5400 1900 2    40   ~ 0
@@
 Connection ~ 8500 1500
 Wire Wire Line
-	9000 1250 9100 1250
-Wire Wire Line
-	9500 1250 9600 1250
-Wire Wire Line
-	9000 1700 9100 1700
-Wire Wire Line
-	9500 1700 9600 1700
+	9000 1250 9600 1250
+Wire Wire Line
+	9000 1700 9600 1700
 Wire Wire Line
 	10000 1250 10100 1250
@@
 Wire Wire Line
 	2450 4950 2450 5600
-Wire Wire Line
-	2450 6100 2350 6100
-Wire Wire Line
-	2350 6100 2350 6200
-Wire Wire Line
-	2450 5700 1300 5700
-Wire Wire Line
-	2450 5800 1050 5800
-Wire Wire Line
-	3550 5750 3650 5750
-Wire Wire Line
-	3650 6000 3550 6000
 $Comp
 L MountingHole U8
@@
 Wire Wire Line
 	1370 4070 1270 4070
-Wire Wire Line
-	4150 6000 4200 6000
-Wire Wire Line
-	4200 6000 4200 5400
-Wire Wire Line
-	4150 5750 4200 5750
-Connection ~ 4200 5750
-Wire Wire Line
-	2350 6200 2300 6200
-Wire Wire Line
-	1650 6200 1800 6200
-Wire Wire Line
-	1050 5800 1050 5700
-Wire Wire Line
-	1300 5200 1050 5200
 Connection ~ 2100 4950
 Wire Wire Line
@@
 Wire Wire Line
 	5470 4110 5470 4050
+Text Label 3550 6000 0    60   ~ 0
+IO5
+Text Label 2450 5700 2    60   ~ 0
+IO23
+$Comp
+L GND #PWR012
+U 1 1 58FDB63D
+P 1950 6000
+F 0 "#PWR012" H 1950 5750 50  0001 C CNN
+F 1 "GND" H 1950 5850 50  0000 C CNN
+F 2 "" H 1950 6000 50  0000 C CNN
+F 3 "" H 1950 6000 50  0000 C CNN
+	1    1950 6000
+	1    0    0    -1
+$EndComp
+Wire Wire Line
+	1950 6000 1950 5800
+Wire Wire Line
+	1950 5800 2450 5800
+Text Label 2450 5900 2    60   ~ 0
+IO18
+Text Label 2450 6000 2    60   ~ 0
+IO19
+NoConn ~ 2450 6100
+NoConn ~ 3550 5750
+$Comp
+L Q_NPN_BEC Q1
+U 1 1 58FE0131
+P 10550 2600
+F 0 "Q1" H 10750 2650 50  0000 L CNN
+F 1 "Q_NPN_BEC" H 10750 2550 50  0000 L CNN
+F 2 "EE:SOT_23" H 10750 2700 50  0001 C CNN
+F 3 "" H 10550 2600 50  0000 C CNN
+	1    10550 2600
+	1    0    0    -1
+$EndComp
+Text Label 5400 2200 2    60   ~ 0
+IO18
+Text Label 5400 2300 2    60   ~ 0
+IO19
+Text Label 5400 2900 2    60   ~ 0
+IO23
+Text Label 5400 2100 2    60   ~ 0
+IO5
+$Comp
+L CONN_01X03 P31
+U 1 1 58FDEC1E
+P 9600 4400
+F 0 "P31" H 9600 4600 50  0000 C CNN
+F 1 "CONN_01X03" V 9700 4400 50  0000 C CNN
+F 2 "Pin_Headers:Pin_Header_Straight_1x03_Pitch2.54mm" H 9600 4400 50  0001 C CNN
+F 3 "" H 9600 4400 50  0000 C CNN
+	1    9600 4400
+	1    0    0    -1
+$EndComp
+$Comp
+L CONN_01X03 P32
+U 1 1 58FDECF4
+P 10000 4400
+F 0 "P32" H 10000 4600 50  0000 C CNN
+F 1 "CONN_01X03" V 10100 4400 50  0000 C CNN
+F 2 "Pin_Headers:Pin_Header_Straight_1x03_Pitch2.54mm" H 10000 4400 50  0001 C CNN
+F 3 "" H 10000 4400 50  0000 C CNN
+	1    10000 4400
+	1    0    0    -1
+$EndComp
+$Comp
+L CONN_01X03 P33
+U 1 1 58FDEDD5
+P 10400 4400
+F 0 "P33" H 10400 4600 50  0000 C CNN
+F 1 "CONN_01X03" V 10500 4400 50  0000 C CNN
+F 2 "Pin_Headers:Pin_Header_Straight_1x03_Pitch2.54mm" H 10400 4400 50  0001 C CNN
+F 3 "" H 10400 4400 50  0000 C CNN
+	1    10400 4400
+	1    0    0    -1
+$EndComp
+$Comp
+L CONN_01X03 P34
+U 1 1 58FDEEB9
+P 10800 4400
+F 0 "P34" H 10800 4600 50  0000 C CNN
+F 1 "CONN_01X03" V 10900 4400 50  0000 C CNN
+F 2 "Pin_Headers:Pin_Header_Straight_1x03_Pitch2.54mm" H 10800 4400 50  0001 C CNN
+F 3 "" H 10800 4400 50  0000 C CNN
+	1    10800 4400
+	1    0    0    -1
+$EndComp
+NoConn ~ 10600 4300
+NoConn ~ 10600 4400
+NoConn ~ 10600 4500
+NoConn ~ 10200 4300
+NoConn ~ 10200 4400
+NoConn ~ 10200 4500
+NoConn ~ 9800 4300
+NoConn ~ 9800 4400
+NoConn ~ 9800 4500
+NoConn ~ 9400 4300
+NoConn ~ 9400 4400
+NoConn ~ 9400 4500
+NoConn ~ 7350 6100
 $EndSCHEMATC

Commit message: v0.3
Connections:
- net GND: no longer U2.3 (CMD)
- net IO23: now also U2.3 (CMD); no longer U2.2 (CD/DATA3)
- net IO5: now also U2.2 (CD/DATA3); no longer U2.1 (DATA2)
Changed lines of the file:
@@
 Wire Wire Line
 	5470 4110 5470 4050
-Text Label 3550 6000 0    60   ~ 0
+Text Label 2450 5700 2    60   ~ 0
 IO5
-Text Label 2450 5700 2    60   ~ 0
+Text Label 2450 5800 2    60   ~ 0
 IO23
-$Comp
-L GND #PWR012
-U 1 1 58FDB63D
-P 1950 6000
-F 0 "#PWR012" H 1950 5750 50  0001 C CNN
-F 1 "GND" H 1950 5850 50  0000 C CNN
-F 2 "" H 1950 6000 50  0000 C CNN
-F 3 "" H 1950 6000 50  0000 C CNN
-	1    1950 6000
-	1    0    0    -1
-$EndComp
-Wire Wire Line
-	1950 6000 1950 5800
-Wire Wire Line
-	1950 5800 2450 5800
 Text Label 2450 5900 2    60   ~ 0
 IO18
