File: Hornbill_PCB/Hornbill.kicad_pcb (KiCad board)
At the start: 2 copper layers, 90 x 60 mm, 69 parts, among them P1 CONN_01X19, P10 CONN_01X03, P11 CONN_01X03, P12 CONN_01X19, P13 CONN_01X03, P14 CONN_01X01, P14 CONN_01X09, P15 CONN_01X09, P16 CONN_01X09, P17 CONN_01X09, P18 CONN_01X09, P19 CONN_01X09, P2 CONN_01X19, P20 CONN_01X09, P21 CONN_01X09, P22 CONN_01X09, P23 CONN_01X09, P24 CONN_01X09, P25 CONN_01X13, P26 CONN_01X13, P27 CONN_01X13, P28 CONN_01X13, P29 CONN_01X09, P3 CONN_01X19, P30 CONN_01X09, P31 CONN_01X03, P32 CONN_01X03, P33 CONN_01X03, P34 CONN_01X03, P4 CONN_01X19, P5 CONN_01X19, P6 CONN_01X19, P7 CONN_01X03, P8 CONN_01X19, P9 CONN_01X03, Q1 Q_NPN_BEC, U2 SD_Crard, U3 RGB_4pin, U4 ESP32_Breakout1, U5 MountingHole, U6 MountingHole, U7 MountingHole, U8 MountingHole

Commit message: v0.3
Connections:
- U2 pad 1: /IO5 -> Net-(U2-Pad1)
- U2 pad 2: /IO23 -> /IO5
- U2 pad 3: GND -> /IO23
Routing:
- net GND: track 193.3 -> 187.3 mm
- net /IO18: track 56.8 -> 54.7 mm
- net /IO5: track 54.6 -> 55.5 mm
Other:
- board text added: "v0.3"
- board text removed: "v0.2"
Changed lines of the file:
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@@
-(kicad_pcb (version 4) (host pcbnew 4.0.4-stable)
+(kicad_pcb (version 4) (host pcbnew 4.0.5)
   (general
-    (links 100)
+    (links 99)
     (no_connects 0)
-    (area 17.150001 17.3 135.742301 114.683181)
+    (area 44.924999 49.924999 135.075001 110.075001)
     (thickness 1.6)
     (drawings 114)
-    (tracks 475)
+    (tracks 468)
     (zones 0)
     (modules 69)
-    (nets 364)
+    (nets 365)
   )
   (page A4)
@@
   (net 362 "Net-(P34-Pad2)")
   (net 363 "Net-(P34-Pad3)")
+  (net 364 "Net-(U2-Pad1)")
   (net_class Default "This is the default net class."
     (clearance 0.15)
@@
     (add_net "Net-(R5-Pad1)")
     (add_net "Net-(RH1-Pad3)")
+    (add_net "Net-(U2-Pad1)")
     (add_net "Net-(U2-Pad8)")
     (add_net "Net-(U2-Pad9)")
@@
     (fp_line (start 2.2 0) (end 8.8 0) (layer F.SilkS) (width 0.15))
     (pad 1 smd rect (at 4.4 -0.8 270) (size 0.7 1.5) (layers F.Cu F.Paste F.Mask)
-      (net 346 /IO5))
+      (net 364 "Net-(U2-Pad1)"))
     (pad 2 smd rect (at 3.3 -0.8 270) (size 0.7 1.5) (layers F.Cu F.Paste F.Mask)
-      (net 347 /IO23))
+      (net 346 /IO5))
     (pad 3 smd rect (at 2.2 -0.8 270) (size 0.7 1.5) (layers F.Cu F.Paste F.Mask)
-      (net 2 GND))
+      (net 347 /IO23))
     (pad 4 smd rect (at 1.1 -0.8 270) (size 0.7 1.5) (layers F.Cu F.Paste F.Mask)
       (net 1 3.3V))
@@
       (xy -3.214253 7.828463)) (layer B.SilkS) (width 0.01))
   )
-  (gr_text v0.2 (at 54.356 63.5 90) (layer B.SilkS)
+  (gr_text v0.3 (at 54.356 63.5 90) (layer B.SilkS)
     (effects (font (size 1.5 1.5) (thickness 0.3)) (justify mirror))
   )
@@
   (segment (start 63.881 74.93) (end 62.865 74.93) (width 0.4) (layer F.Cu) (net 2))
   (segment (start 64.4144 74.3966) (end 63.881 74.93) (width 0.4) (layer F.Cu) (net 2))
-  (segment (start 60.236 64.176) (end 65.11 64.176) (width 0.4) (layer F.Cu) (net 2))
-  (segment (start 65.466 63.82) (end 65.466 63.119) (width 0.4) (layer F.Cu) (net 2))
-  (segment (start 65.11 64.176) (end 65.466 63.82) (width 0.4) (layer F.Cu) (net 2))
   (segment (start 65.466 60.96) (end 65.466 60.005) (width 0.4) (layer F.Cu) (net 2))
   (segment (start 61.679 60.876) (end 60.236 60.876) (width 0.4) (layer F.Cu) (net 2))
@@
   (segment (start 63.754 71.12) (end 63.754 71.628) (width 0.4) (layer F.Cu) (net 345))
   (segment (start 63.974 70.9) (end 63.754 71.12) (width 0.4) (layer F.Cu) (net 345))
-  (segment (start 105.41 68.58) (end 105.41 70.866) (width 0.25) (layer F.Cu) (net 346))
-  (segment (start 61.55 66.376) (end 60.236 66.376) (width 0.25) (layer F.Cu) (net 346))
-  (segment (start 64.643 69.469) (end 61.55 66.376) (width 0.25) (layer F.Cu) (net 346))
-  (segment (start 72.898 69.469) (end 64.643 69.469) (width 0.25) (layer F.Cu) (net 346))
-  (segment (start 72.898 69.469) (end 72.898 69.469) (width 0.25) (layer F.Cu) (net 346))
-  (segment (start 78.867 69.469) (end 72.898 69.469) (width 0.25) (layer F.Cu) (net 346))
-  (segment (start 82.042 72.644) (end 78.867 69.469) (width 0.25) (layer F.Cu) (net 346))
-  (segment (start 103.632 72.644) (end 82.042 72.644) (width 0.25) (layer F.Cu) (net 346))
-  (segment (start 105.41 70.866) (end 103.632 72.644) (width 0.25) (layer F.Cu) (net 346))
+  (segment (start 105.41 68.58) (end 105.41 71.628) (width 0.25) (layer F.Cu) (net 346) (status 400000))
+  (segment (start 61.339 65.276) (end 60.236 65.276) (width 0.25) (layer F.Cu) (net 346) (status 800000))
+  (segment (start 65.659 69.596) (end 61.339 65.276) (width 0.25) (layer F.Cu) (net 346))
+  (segment (start 78.994 69.596) (end 65.659 69.596) (width 0.25) (layer F.Cu) (net 346))
+  (segment (start 82.042 72.644) (end 78.994 69.596) (width 0.25) (layer F.Cu) (net 346))
+  (segment (start 104.394 72.644) (end 82.042 72.644) (width 0.25) (layer F.Cu) (net 346))
+  (segment (start 105.41 71.628) (end 104.394 72.644) (width 0.25) (layer F.Cu) (net 346))
   (segment (start 105.41 68.58) (end 105.41 64.77) (width 1) (layer F.Cu) (net 346))
-  (segment (start 66.04 66.548) (end 63.246 66.548) (width 0.25) (layer B.Cu) (net 347))
-  (segment (start 78.359 67.818) (end 75.565 65.024) (width 0.25) (layer B.Cu) (net 347))
-  (segment (start 75.565 65.024) (end 69.342 65.024) (width 0.25) (layer B.Cu) (net 347))
-  (segment (start 69.342 65.024) (end 67.818 66.548) (width 0.25) (layer B.Cu) (net 347))
-  (segment (start 67.818 66.548) (end 66.04 66.548) (width 0.25) (layer B.Cu) (net 347))
-  (segment (start 78.359 68.707) (end 78.359 67.818) (width 0.25) (layer B.Cu) (net 347))
-  (segment (start 61.974 65.276) (end 60.236 65.276) (width 0.25) (layer F.Cu) (net 347))
-  (segment (start 62.611 65.913) (end 61.974 65.276) (width 0.25) (layer F.Cu) (net 347))
-  (via (at 62.611 65.913) (size 0.91) (drill 0.5) (layers F.Cu B.Cu) (net 347))
-  (segment (start 63.246 66.548) (end 62.611 65.913) (width 0.25) (layer B.Cu) (net 347))
-  (segment (start 85.09 68.58) (end 85.09 73.533) (width 0.25) (layer B.Cu) (net 347))
-  (segment (start 78.359 72.39) (end 78.359 68.707) (width 0.25) (layer B.Cu) (net 347))
-  (segment (start 78.359 68.707) (end 78.359 68.58) (width 0.25) (layer B.Cu) (net 347))
-  (segment (start 80.645 74.676) (end 78.359 72.39) (width 0.25) (layer B.Cu) (net 347))
-  (segment (start 83.947 74.676) (end 80.645 74.676) (width 0.25) (layer B.Cu) (net 347))
-  (segment (start 85.09 73.533) (end 83.947 74.676) (width 0.25) (layer B.Cu) (net 347))
+  (segment (start 62.611 65.532) (end 62.611 65.151) (width 0.25) (layer B.Cu) (net 347))
+  (segment (start 85.09 72.136) (end 83.058 74.168) (width 0.25) (layer B.Cu) (net 347))
+  (segment (start 83.058 74.168) (end 80.01 74.168) (width 0.25) (layer B.Cu) (net 347))
+  (segment (start 80.01 74.168) (end 78.359 72.517) (width 0.25) (layer B.Cu) (net 347))
+  (segment (start 78.359 72.517) (end 78.359 67.564) (width 0.25) (layer B.Cu) (net 347))
+  (segment (start 78.359 67.564) (end 75.565 64.77) (width 0.25) (layer B.Cu) (net 347))
+  (segment (start 75.565 64.77) (end 66.548 64.77) (width 0.25) (layer B.Cu) (net 347))
+  (segment (start 66.548 64.77) (end 64.897 66.421) (width 0.25) (layer B.Cu) (net 347))
+  (segment (start 64.897 66.421) (end 63.5 66.421) (width 0.25) (layer B.Cu) (net 347))
+  (segment (start 63.5 66.421) (end 62.611 65.532) (width 0.25) (layer B.Cu) (net 347))
+  (segment (start 85.09 68.58) (end 85.09 72.136) (width 0.25) (layer B.Cu) (net 347) (status 400000))
+  (segment (start 61.636 64.176) (end 60.236 64.176) (width 0.25) (layer F.Cu) (net 347) (status 800000))
+  (segment (start 62.484 65.024) (end 61.636 64.176) (width 0.25) (layer F.Cu) (net 347))
+  (via (at 62.484 65.024) (size 0.91) (drill 0.5) (layers F.Cu B.Cu) (net 347))
+  (segment (start 62.611 65.151) (end 62.484 65.024) (width 0.25) (layer B.Cu) (net 347))
   (segment (start 85.09 68.58) (end 85.09 64.77) (width 1) (layer F.Cu) (net 347))
   (segment (start 67.437 68.961) (end 66.675 68.961) (width 0.25) (layer F.Cu) (net 348))
@@
   (segment (start 73.152 68.961) (end 73.152 68.961) (width 0.25) (layer F.Cu) (net 348))
   (segment (start 73.152 68.961) (end 67.437 68.961) (width 0.25) (layer F.Cu) (net 348))
-  (segment (start 67.437 68.961) (end 65.405 68.961) (width 0.25) (layer F.Cu) (net 348))
   (segment (start 102.87 68.58) (end 102.87 71.12) (width 0.25) (layer F.Cu) (net 348))
   (segment (start 61.976 61.976) (end 60.236 61.976) (width 0.25) (layer F.Cu) (net 348))

Commit message: v0.3
Routing:
- net 3.3V: track 108.5 -> 109.1 mm
Changed lines of the file:
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@@
     (links 99)
     (no_connects 0)
-    (area 44.924999 49.924999 135.075001 110.075001)
+    (area 17.150001 17.3 135.742301 114.683181)
     (thickness 1.6)
     (drawings 114)
-    (tracks 468)
+    (tracks 470)
     (zones 0)
     (modules 69)
@@
     (add_net "Net-(U2-Pad9)")
   )
+  (module ee:RGB_SMD_4pin_New (layer F.Cu)
+    (at 69.088 56.388 180)
+    (fp_text reference U3 (at -0.1016 -1.4732 180) (layer F.SilkS)
+      (effects (font (size 0.635 0.635) (thickness 0.15)))
+    )
+    (fp_text value RGB_4pin (at 0 2.6 180) (layer F.SilkS) hide
+      (effects (font (size 1 1) (thickness 0.15)))
+    )
+    (fp_line (start -0.75 0.5) (end -0.75 -0.75) (layer F.SilkS) (width 0.15))
+    (fp_line (start -0.75 -0.75) (end 0.75 -0.75) (layer F.SilkS) (width 0.15))
+    (fp_line (start 0.75 -0.75) (end 0.75 0) (layer F.SilkS) (width 0.15))
+    (fp_line (start 0.75 0) (end 0.25 0.5) (layer F.SilkS) (width 0.15))
+    (fp_line (start 0.25 0.5) (end -0.75 0.5) (layer F.SilkS) (width 0.15))
+    (pad 1 smd rect (at -1.45 0.7125 180) (size 1 0.8) (layers F.Cu F.Paste F.Mask)
+      (net 1 3.3V))
+    (pad 2 smd rect (at 1.45 0.7125 180) (size 1 0.8) (layers F.Cu F.Paste F.Mask)
+      (net 119 "Net-(R14-Pad1)"))
+    (pad 3 smd rect (at -1.45 -0.7125 180) (size 1 0.8) (layers F.Cu F.Paste F.Mask)
+      (net 117 "Net-(R12-Pad1)"))
+    (pad 4 smd rect (at 1.45 -0.7125 180) (size 1 0.8) (layers F.Cu F.Paste F.Mask)
+      (net 118 "Net-(R13-Pad1)"))
+  )
   (module ee:ESP32_Breakout (layer F.Cu)
     (at 105.41 78.74 270)
@@
     )
   )
-  (module ee:RGB_SMD_4pin_New (layer F.Cu)
-    (at 69.088 56.388 180)
-    (fp_text reference U3 (at -0.1016 -1.4732 180) (layer F.SilkS)
-      (effects (font (size 0.635 0.635) (thickness 0.15)))
-    )
-    (fp_text value RGB_4pin (at 0 2.6 180) (layer F.SilkS) hide
-      (effects (font (size 1 1) (thickness 0.15)))
-    )
-    (fp_line (start -1.4478 -0.6858) (end -1.4478 0.7366) (layer F.SilkS) (width 0.15))
-    (fp_line (start -1.4478 0.7366) (end 0.9144 0.7366) (layer F.SilkS) (width 0.15))
-    (fp_line (start 0.9144 0.7366) (end 1.3716 0.2794) (layer F.SilkS) (width 0.15))
-    (fp_line (start 1.3716 0.2794) (end 1.3716 -0.6604) (layer F.SilkS) (width 0.15))
-    (fp_line (start 1.3716 -0.6604) (end -1.4732 -0.6604) (layer F.SilkS) (width 0.15))
-    (pad 1 smd rect (at -1.45 0.7125 180) (size 1 0.8) (layers F.Cu F.Paste F.Mask)
-      (net 1 3.3V))
-    (pad 2 smd rect (at 1.45 0.7125 180) (size 1 0.8) (layers F.Cu F.Paste F.Mask)
-      (net 119 "Net-(R14-Pad1)"))
-    (pad 3 smd rect (at -1.45 -0.7125 180) (size 1 0.8) (layers F.Cu F.Paste F.Mask)
-      (net 117 "Net-(R12-Pad1)"))
-    (pad 4 smd rect (at 1.45 -0.7125 180) (size 1 0.8) (layers F.Cu F.Paste F.Mask)
-      (net 118 "Net-(R13-Pad1)"))
-  )
   (module Pin_Headers:Pin_Header_Straight_1x09_Pitch2.54mm (layer F.Cu)
     (at 85.09 107.95 270)
@@
     (arrow2b (pts (xy 45 30) (xy 46.126504 29.413579)))
   )
-  (segment (start 58.3692 64.0588) (end 58.3692 63.5762) (width 0.4) (layer B.Cu) (net 1))
-  (segment (start 67.9958 56.769) (end 69.088 55.6768) (width 0.4) (layer B.Cu) (net 1))
-  (segment (start 60.071 56.769) (end 67.9958 56.769) (width 0.4) (layer B.Cu) (net 1))
-  (segment (start 57.912 58.928) (end 60.071 56.769) (width 0.4) (layer B.Cu) (net 1))
-  (segment (start 57.912 63.119) (end 57.912 58.928) (width 0.4) (layer B.Cu) (net 1))
+  (segment (start 71.5772 58.166) (end 71.5772 57.7342) (width 0.25) (layer B.Cu) (net 1))
+  (segment (start 79.756 58.1152) (end 79.248 58.6232) (width 0.254) (layer F.Cu) (net 1))
+  (via (at 79.756 58.1152) (size 0.889) (drill 0.635) (layers F.Cu B.Cu) (net 1))
+  (segment (start 78.1812 58.1152) (end 79.756 58.1152) (width 0.254) (layer B.Cu) (net 1))
+  (segment (start 78.1304 58.166) (end 78.1812 58.1152) (width 0.254) (layer B.Cu) (net 1))
+  (segment (start 71.5772 58.166) (end 78.1304 58.166) (width 0.254) (layer B.Cu) (net 1))
+  (segment (start 78.062 58.6232) (end 79.248 58.6232) (width 0.254) (layer F.Cu) (net 1))
+  (segment (start 71.5772 57.7342) (end 69.215 55.372) (width 0.25) (layer B.Cu) (net 1))
+  (segment (start 70.538 55.6755) (end 69.5185 55.6755) (width 0.4) (layer F.Cu) (net 1) (status 400000))
+  (segment (start 69.5185 55.6755) (end 69.215 55.372) (width 0.4) (layer F.Cu) (net 1))
+  (via (at 69.215 55.372) (size 0.91) (drill 0.5) (layers F.Cu B.Cu) (net 1))
+  (segment (start 67.818 56.769) (end 66.167 56.769) (width 0.4) (layer B.Cu) (net 1))
   (segment (start 58.3692 63.5762) (end 57.912 63.119) (width 0.4) (layer B.Cu) (net 1))
+  (segment (start 57.912 63.119) (end 57.912 58.928) (width 0.4) (layer B.Cu) (net 1))
+  (segment (start 57.912 58.928) (end 60.071 56.769) (width 0.4) (layer B.Cu) (net 1))
+  (segment (start 60.071 56.769) (end 66.167 56.769) (width 0.4) (layer B.Cu) (net 1))
+  (segment (start 58.3692 64.0588) (end 58.3692 63.5762) (width 0.4) (layer B.Cu) (net 1))
+  (segment (start 69.215 55.372) (end 67.818 56.769) (width 0.4) (layer B.Cu) (net 1))
   (segment (start 63.566 63.119) (end 63.566 60.96) (width 0.4) (layer F.Cu) (net 1))
   (segment (start 60.236 63.076) (end 63.523 63.076) (width 0.4) (layer F.Cu) (net 1))
   (segment (start 63.523 63.076) (end 63.566 63.119) (width 0.4) (layer F.Cu) (net 1))
-  (segment (start 70.538 55.6755) (end 69.0893 55.6755) (width 0.254) (layer F.Cu) (net 1))
-  (segment (start 69.0893 55.6755) (end 69.088 55.6768) (width 0.254) (layer F.Cu) (net 1))
-  (via (at 69.088 55.6768) (size 0.889) (drill 0.635) (layers F.Cu B.Cu) (net 1))
-  (segment (start 79.248 58.6232) (end 78.062 58.6232) (width 0.254) (layer F.Cu) (net 1))
-  (segment (start 69.088 55.6768) (end 71.5772 58.166) (width 0.254) (layer B.Cu) (net 1))
-  (segment (start 71.5772 58.166) (end 78.1304 58.166) (width 0.254) (layer B.Cu) (net 1))
-  (segment (start 78.1304 58.166) (end 78.1812 58.1152) (width 0.254) (layer B.Cu) (net 1))
-  (segment (start 78.1812 58.1152) (end 79.756 58.1152) (width 0.254) (layer B.Cu) (net 1))
-  (via (at 79.756 58.1152) (size 0.889) (drill 0.635) (layers F.Cu B.Cu) (net 1))
-  (segment (start 79.756 58.1152) (end 79.248 58.6232) (width 0.254) (layer F.Cu) (net 1))
   (segment (start 82.55 91.44) (end 82.55 84.328) (width 0.7) (layer F.Cu) (net 1))
   (segment (start 59.352 63.076) (end 60.236 63.076) (width 0.254) (layer F.Cu) (net 1))
@@
   (segment (start 63.754 71.12) (end 63.754 71.628) (width 0.4) (layer F.Cu) (net 345))
   (segment (start 63.974 70.9) (end 63.754 71.12) (width 0.4) (layer F.Cu) (net 345))
-  (segment (start 105.41 68.58) (end 105.41 71.628) (width 0.25) (layer F.Cu) (net 346) (status 400000))
-  (segment (start 61.339 65.276) (end 60.236 65.276) (width 0.25) (layer F.Cu) (net 346) (status 800000))
+  (segment (start 105.41 68.58) (end 105.41 71.628) (width 0.25) (layer F.Cu) (net 346))
+  (segment (start 61.339 65.276) (end 60.236 65.276) (width 0.25) (layer F.Cu) (net 346))
   (segment (start 65.659 69.596) (end 61.339 65.276) (width 0.25) (layer F.Cu) (net 346))
   (segment (start 78.994 69.596) (end 65.659 69.596) (width 0.25) (layer F.Cu) (net 346))
@@
   (segment (start 64.897 66.421) (end 63.5 66.421) (width 0.25) (layer B.Cu) (net 347))
   (segment (start 63.5 66.421) (end 62.611 65.532) (width 0.25) (layer B.Cu) (net 347))
-  (segment (start 85.09 68.58) (end 85.09 72.136) (width 0.25) (layer B.Cu) (net 347) (status 400000))
-  (segment (start 61.636 64.176) (end 60.236 64.176) (width 0.25) (layer F.Cu) (net 347) (status 800000))
+  (segment (start 85.09 68.58) (end 85.09 72.136) (width 0.25) (layer B.Cu) (net 347))
+  (segment (start 61.636 64.176) (end 60.236 64.176) (width 0.25) (layer F.Cu) (net 347))
   (segment (start 62.484 65.024) (end 61.636 64.176) (width 0.25) (layer F.Cu) (net 347))
   (via (at 62.484 65.024) (size 0.91) (drill 0.5) (layers F.Cu B.Cu) (net 347))
